Commit message: updating

File: mecannum_base_description/urdf/common_properties.xacro (robot description, xacro)
@@ -7,3 +7,21 @@
         <color rgba="0.5 0.5 0.5 1" />
     </material>
+    <xacro:macro name="box_inertia" params="m l w h xyz rpy">
+        <inertial>
+            <origin xyz="${xyz}" rpy="${rpy}" />
+            <mass value="${m}" />
+            <inertia ixx="${(m/12.0) * (h*h + l*l)}" ixy="0" ixz="0"
+                     iyy="${(m/12.0) * (w*w + l*l)}" iyz="0"
+                     izz="${(m/12.0) * (w*w + h*h)}" />
+        </inertial>
+    </xacro:macro>
+    <xacro:macro name="wheel_inertia" params="m r h xyz rpy">
+        <inertial>
+            <origin xyz="${xyz}" rpy="${rpy}"/>
+            <mass value="${m}" />
+            <inertia ixx="${(m/12.0)*(3*r*r + h*h)}" ixy="0" ixz="0"
+                     iyy="${(m/12.0)*(3*r*r + h*h)}" iyz="0"
+                     izz="${((m/2)*r*r)}" />
+        </inertial>
+    </xacro:macro>
 </robot>

File: mecannum_base_description/urdf/mecannum_base.xacro (robot description, xacro)
@@ -15,4 +15,12 @@
             <material name="blue" />
         </visual>
+        <collision>
+            <geometry>
+                <box size="${base_length} ${base_width} ${base_height}" />
+            </geometry>
+            <origin xyz="0 0 ${base_height / 2.0}" rpy="0 0 0" />
+        </collision>
+        <xacro:box_inertia m="7.0" l="${base_length}" w="${base_width}" h="${base_height}"
+                           xyz="0 0 ${base_height / 2.0}" rpy="0 0 0" />
     </link>
     <joint name="base_footprint_base_link_joint" type="fixed">
@@ -23,10 +31,10 @@
     <xacro:macro name="wheel_link" params="prefix mesh_filename is_left">
         <link name="${prefix}_wheel_link">
+            <xacro:property name="y_offset" value="0" />
             <visual>
                 <geometry>
-                    <mesh filename="package://mecannum_base_description/meshes/${mesh_filename}" scale="0.00133 0.00133 0.00092"/>
+                    <mesh filename="${mesh_filename}" scale="0.00133 0.00133 0.00092"/>
                 </geometry>
                 <!-- Define a temporary variable for adjusting the origin -->
-                <xacro:property name="y_offset" value="0" />
                 <xacro:if value="${is_left}">
                     <xacro:property name="y_offset" value="${-(base_width - wheel_length) / 2.0}" />
@@ -35,7 +43,18 @@
                 <material name="grey" />
             </visual>
+            <collision>
+                <geometry>
+                    <mesh filename="${mesh_filename}" scale="0.00133 0.00133 0.00092"/>
+                </geometry>
+                <!-- Define a temporary variable for adjusting the origin -->
+                <xacro:if value="${is_left}">
+                    <xacro:property name="y_offset" value="${-(base_width - wheel_length) / 2.0}" />
+                </xacro:if>
+                <origin xyz="0 ${y_offset} 0" rpy="${pi / 2} 0 0" />
+            </collision>
+            <xacro:wheel_inertia m="0.5" r="${wheel_radius}" h="${wheel_length}" xyz="0 ${y_offset} 0" rpy="${pi / 2} 0 0" />
         </link>
     </xacro:macro>
-    <xacro:wheel_link prefix="rear_right" mesh_filename="Mecannum_Wheel_Left.stl" is_left="true" />
+    <xacro:wheel_link prefix="rear_right" mesh_filename="file://$(find mecannum_base_description)/meshes/Mecannum_Wheel_Left.stl" is_left="true" />
     <joint name="base_rear_right_wheel_joint" type="continuous">
         <parent link="base_link" />
@@ -44,5 +63,5 @@
         <axis xyz="0 1 0" />
     </joint>
-    <xacro:wheel_link prefix="rear_left" mesh_filename="Mecannum_Wheel_Right.stl" is_left="false" />
+    <xacro:wheel_link prefix="rear_left" mesh_filename="file://$(find mecannum_base_description)/meshes/Mecannum_Wheel_Right.stl" is_left="false" />
     <joint name="base_rear_left_wheel_joint" type="continuous">
         <parent link="base_link" />
@@ -51,5 +70,5 @@
         <axis xyz="0 1 0" />
     </joint>
-    <xacro:wheel_link prefix="front_right" mesh_filename="Mecannum_Wheel_Right.stl" is_left="false" />
+    <xacro:wheel_link prefix="front_right" mesh_filename="file://$(find mecannum_base_description)/meshes/Mecannum_Wheel_Right.stl" is_left="false" />
     <joint name="base_front_right_wheel_joint" type="continuous">
         <parent link="base_link" />
@@ -58,5 +77,5 @@
         <axis xyz="0 1 0" />
     </joint>
-    <xacro:wheel_link prefix="front_left" mesh_filename="Mecannum_Wheel_Left.stl" is_left="true" />
+    <xacro:wheel_link prefix="front_left" mesh_filename="file://$(find mecannum_base_description)/meshes/Mecannum_Wheel_Left.stl" is_left="true" />
     <joint name="base_front_left_wheel_joint" type="continuous">
         <parent link="base_link" />

File: mecannum_base_description/urdf/my_robot.xacro (robot description, xacro)
@@ -3,3 +3,4 @@
     <xacro:include filename="common_properties.xacro" />
     <xacro:include filename="mecannum_base.xacro" />
+    <xacro:include filename="mecannum_base_gazebo.xacro" />
 </robot>
